File: PCB/controller/_autosave-controller.kicad_sch (KiCad schematic)
At the start: 32 parts, among them J1 USB_C_Receptacle_USB2.0_16P, Q5 BSS138, SW2 SW_Push, SW3 SW_Push, U1 NanoS3, U2 COM-09032, U3 TPS61200DRC

Commit message: Refactor code structure for improved readability and maintainability
Connections:
- net BOOT: now also U1.29 (IO0); no longer U1.30 (IO33)
- net LED_LV: now also U1.23 (IO35); no longer U1.15 (IO14)
