File: PCB/controller/controller.kicad_pcb (KiCad board)
At the start: 2 copper layers, 13 parts, among them P1 USB_C_Plug_USB2.0, SW1 SW_Push, SW2 SW_Push, SW3 SW_Push, U1 NanoS3, U2 COM-09032

Commit message: sadasd
Parts:
- removed P1: USB_C_Plug_USB2.0, Connector_USB:USB_C_Receptacle_G-Switch_GT-USB-7025
- removed SW1: SW_Push, Button_Switch_SMD:SW_Push_SPST_NO_Alps_SKRK
- added BOOT: SW_Push, Button_Switch_SMD:SW_Push_SPST_NO_Alps_SKRK, B.Cu at (160.1, 27.5)
- added D4: D_Shockley, Diode_SMD:D_SMA-SMB_Universal_Handsoldering, B.Cu at (158.0, 39.0)
- added J1: USB_C_Receptacle_USB2.0_16P, Connector_USB:USB_C_Receptacle_XKB_U262-16XN-4BVC11, F.Cu at (170.8, 19.8)
- added R2: R5.1kΩ, Resistor_SMD:R_0201_0603Metric_Pad0.64x0.40mm_HandSolder, B.Cu at (173.1, 24.9)
- added RESET: SW_Push, Button_Switch_SMD:SW_Push_SPST_NO_Alps_SKRK, B.Cu at (161.0, 44.0)
- BT1, C1, C2, R1: moved to B.Cu
- D2, D3: footprint LED_SMD:LED_SK6812MINI_PLCC4_3.5x3.5mm_P1.75mm -> footprints:SK6812MINI-E; moved to B.Cu
- U1: footprint footprints:NanoS3 -> NanoS3:NanoS3_HandSolder; moved to F.Cu
- moved BT1 171.0 mm to (201.4, 22.5), turned to 90 degrees
- moved C2 144.4 mm to (194.1, 41.1), turned to 180 degrees
- moved D2 136.3 mm to (175.0, 38.2), turned to 180 degrees
- moved R1 130.5 mm to (168.1, 24.9)
- moved C1 117.5 mm to (175.0, 41.0), turned to 180 degrees
- moved D1 116.6 mm to (164.5, 48.5), turned to 180 degrees
- moved D3 76.6 mm to (194.1, 38.5), turned to 180 degrees
- moved SW3 76.4 mm to (194.1, 34.0)
- moved U2 67.4 mm to (140.0, 34.0)
- moved U1 60.9 mm to (158.0, 33.8), turned to 90 degrees
- moved SW2 48.3 mm to (175.0, 34.0)
Connections:
- R1 pad 2: Net-(P1-CC) -> /CC2
- U1 pad 12: SEL -> DIR_H
- U1 pad 13: DIR_H -> DIR_V
- U1 pad 14: DIR_V -> SEL
- U1 pad 30: unconnected-(U1-IO33-Pad30) -> BOOT
- U1 pad 8: unconnected-(U1-3v3-Pad8) -> 3.3V
- U2 pad H1: VBUS -> 3.3V
- U2 pad V1: VBUS -> 3.3V
Routing:
- net VBAT: track 0.00 -> 58.0 mm, vias 0 -> 3
- net USE: track 0.00 -> 52.0 mm
- net D-: track 0.00 -> 33.0 mm, vias 0 -> 2
- net 3.3V: track 0.00 -> 32.0 mm
- net D+: track 0.00 -> 31.6 mm, vias 0 -> 2
- net DASH: track 0.00 -> 29.2 mm
- net Net-(D4-A): track 0.00 -> 28.3 mm, vias 0 -> 1
- net DIR_V: track 0.00 -> 22.1 mm
- net SEL: track 0.00 -> 21.0 mm
- net VBUS: track 0.00 -> 15.6 mm, vias 0 -> 1
- net Net-(D2-DOUT): track 0.00 -> 14.6 mm
- net DIR_H: track 0.00 -> 13.4 mm
- net BOOT: track 0.00 -> 7.29 mm, vias 0 -> 1
- net Net-(U1-RESET): track 0.00 -> 3.82 mm, vias 0 -> 1
- net STAT: track 0.00 -> 2.06 mm
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- added copper zone on B.Cu, net GND
- added copper zone on F.Cu, net GND
Other:
- board outline added: 79 x 33 mm

Commit message: Add lock files for PCB controller and schematic with user information
Parts:
- added R3: 120Ω, Capacitor_SMD:C_0603_1608Metric_Pad1.08x0.95mm_HandSolder, B.Cu at (166.0, 47.5)
- D1: footprint LED_SMD:LED_0201_0603Metric_Pad0.64x0.40mm_HandSolder -> LED_SMD:LED_0603_1608Metric_Pad1.05x0.95mm_HandSolder; moved to B.Cu
- R1, R2: footprint Resistor_SMD:R_0201_0603Metric_Pad0.64x0.40mm_HandSolder -> Resistor_SMD:R_0603_1608Metric_Pad0.98x0.95mm_HandSolder
- moved R2 5.05 mm to (172.0, 20.0), turned to -90 degrees
- moved R1 5.02 mm to (169.0, 20.0), turned to -90 degrees
- moved D1 3.35 mm to (166.0, 45.5), turned to 0 degrees
- moved C2 0.20 mm to (194.1, 41.3)
- renumbered BOOT to SW_BOOT1, RESET to SW_RESET1
Connections:
- D1 pad 2: STAT -> Net-(D1-A)
- U1 pad 27: unconnected-(U1-IO9-Pad27) -> STAT
Routing:
- net VBUS: track 15.6 -> 51.9 mm, vias 1 -> 3
- net STAT: track 2.06 -> 14.2 mm, vias 0 -> 3
- net Net-(J1-CC1): track 2.06 -> 5.52 mm
- net /CC2: track 2.06 -> 5.52 mm
- net Net-(D1-A): track 0.00 -> 2.01 mm
- net GND: track 1.54 -> 0.00 mm, vias 4 -> 3
- net D-: track 33.0 -> 32.2 mm

Commit message: Refactor code structure for improved readability and maintainability
Parts:
- added C3: 10uF, Capacitor_SMD:C_0603_1608Metric_Pad1.08x0.95mm_HandSolder, B.Cu at (129.0, 22.5)
- added C4: 22uF, Capacitor_SMD:C_0603_1608Metric_Pad1.08x0.95mm_HandSolder, B.Cu at (145.5, 22.5)
- added C5: 0.1uF, Capacitor_SMD:C_0603_1608Metric_Pad1.08x0.95mm_HandSolder, B.Cu at (135.5, 19.5)
- added D5: D_Shockley, Diode_SMD:D_SMA-SMB_Universal_Handsoldering, B.Cu at (154.0, 31.5)
- added L1: 2.2µH/±20%/1.5A, Inductor_SMD:L_1008_2520Metric_Pad1.43x2.20mm_HandSolder, B.Cu at (140.0, 24.3)
- added Q5: BSS138, Package_TO_SOT_SMD:SOT-23, B.Cu at (170.6, 42.1)
- added R10: 1.8M, Resistor_SMD:R_0603_1608Metric_Pad0.98x0.95mm_HandSolder, B.Cu at (141.5, 19.6)
- added R11: 200k, Resistor_SMD:R_0603_1608Metric_Pad0.98x0.95mm_HandSolder, B.Cu at (139.5, 19.6)
- added R4: 10K, Resistor_SMD:R_0603_1608Metric_Pad0.98x0.95mm_HandSolder, B.Cu at (170.5, 45.0)
- added R5: 10K, Resistor_SMD:R_0603_1608Metric_Pad0.98x0.95mm_HandSolder, B.Cu at (169.8, 39.0)
- added R6: 10kΩ, Resistor_SMD:R_0603_1608Metric_Pad0.98x0.95mm_HandSolder, B.Cu at (149.3, 36.2)
- added R7: 15kΩ, Resistor_SMD:R_0603_1608Metric_Pad0.98x0.95mm_HandSolder, B.Cu at (147.8, 36.2)
- added R8: 100kΩ, Resistor_SMD:R_0603_1608Metric_Pad0.98x0.95mm_HandSolder, B.Cu at (174.5, 29.5)
- added R9: 100kΩ, Resistor_SMD:R_0603_1608Metric_Pad0.98x0.95mm_HandSolder, B.Cu at (174.5, 27.5)
- added U3: TPS61200DRC, Package_SON:Texas_S-PVSON-N10_ThermalVias, B.Cu at (132.8, 22.6)
- moved BT1 1.56 mm to (203.0, 22.5)
Connections:
- D2 pad 3: LED -> LED_HV
- D4 pad 2: Net-(D4-A) -> +5V
- J1 pad A4: Net-(D4-A) -> +5V
- J1 pad A9: Net-(D4-A) -> +5V
- J1 pad B4: Net-(D4-A) -> +5V
- J1 pad B9: Net-(D4-A) -> +5V
- U1 pad 12: DIR_H -> SEL
- U1 pad 13: DIR_V -> 5V_SENSE
- U1 pad 14: SEL -> BOOST_EN
- U1 pad 21: unconnected-(U1-IO6-Pad21) -> DIR_H
- U1 pad 22: unconnected-(U1-IO5-Pad22) -> DIR_V
- U1 pad 23: unconnected-(U1-IO35-Pad23) -> LED_LV
- U1 pad 29: unconnected-(U1-IO0-Pad29) -> BOOT
- U1 pad 30: BOOT -> unconnected-(U1-IO33-Pad30)
- U1 pad 33: unconnected-(U1-IO1-Pad33) -> BAT_SENSE
- U1 pad 4: VBUS -> +5V
Routing:
- net VBAT: track 58.0 -> 106.0 mm, vias 3 -> 5
- net +5V: track 0.00 -> 46.5 mm, vias 0 -> 2
- net Net-(D4-A): track 28.3 -> 0.00 mm, vias 1 -> 0
- net BOOST_EN: track 0.00 -> 26.4 mm, vias 0 -> 1
- net +5V_Boost: track 0.00 -> 24.8 mm
- net Net-(U3-FB): track 0.00 -> 11.7 mm
- net BAT_SENSE: track 0.00 -> 11.4 mm, vias 0 -> 1
- net LED_LV: track 0.00 -> 8.68 mm, vias 0 -> 1
- net DIR_H: track 13.4 -> 20.8 mm
- net Net-(U3-L): track 0.00 -> 6.49 mm
- net 5V_SENSE: track 0.00 -> 4.15 mm, vias 0 -> 1
- net LED_HV: track 0.00 -> 3.91 mm
- net STAT: track 14.2 -> 16.8 mm
- net DIR_V: track 22.1 -> 24.5 mm
- net GND: track 0.00 -> 2.16 mm, vias 3 -> 4
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