File: PCB/controller/controller.kicad_pcb (KiCad board)
At the start: 2 copper layers, 79 x 33 mm, 32 parts, among them J1 USB_C_Receptacle_USB2.0_16P, Q5 BSS138, SW2 SW_Push, SW3 SW_Push, U1 NanoS3, U2 COM-09032, U3 TPS61200DRC

Commit message: Add production files for PCB controller design
- Created designators.csv with component designators and their counts.
- Added netlist.ipc containing detailed netlist information for PCB connections.
- Introduced positions.csv to specify component positions, rotations, and layers on the PCB.
Parts:
- C1, C2: value C -> 0.1uF
- C5: footprint Capacitor_SMD:C_0603_1608Metric_Pad1.08x0.95mm_HandSolder -> Capacitor_SMD:C_0805_2012Metric_Pad1.18x1.45mm_HandSolder
- moved BT1 2.13 mm to (201.6, 24.1)
- moved C5 1.36 mm to (136.8, 19.9)
- moved C1 0.95 mm to (175.0, 42.0)
- moved D2 0.95 mm to (175.0, 39.2)
- moved Q5 0.95 mm to (170.6, 43.0)
- moved R4 0.95 mm to (170.5, 46.0)
- moved R5 0.95 mm to (169.8, 40.0)
- moved C2 0.70 mm to (194.1, 42.0)
- moved D3 0.70 mm to (194.1, 39.2)
Routing:
- net USE: track 52.0 -> 54.5 mm
- net VBAT: track 106.0 -> 103.6 mm
- net D-: track 32.2 -> 33.2 mm
- net VBUS: track 54.0 -> 53.1 mm
- net +5V: track 46.5 -> 45.9 mm

Commit message: Add lock file for PCB controller with hostname and username information
Parts:
- C5: footprint Capacitor_SMD:C_0805_2012Metric_Pad1.18x1.45mm_HandSolder -> Capacitor_SMD:C_0603_1608Metric_Pad1.08x0.95mm_HandSolder
- J1: footprint Connector_USB:USB_C_Receptacle_XKB_U262-16XN-4BVC11 -> Connector_USB:USB_C_Receptacle_G-Switch_GT-USB-7010ASV
- R1, R2: value R5.1kΩ -> R5.1k
- R3: value 120Ω -> 120
- R6: value 10kΩ -> 10k
- R7: value 15kΩ -> 15k
- R8, R9: value 100kΩ -> 100k
Changed lines of the file:
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@@
 		)
 	)
-	(footprint "Connector_USB:USB_C_Receptacle_XKB_U262-16XN-4BVC11"
+	(footprint "Connector_USB:USB_C_Receptacle_G-Switch_GT-USB-7010ASV"
 		(layer "F.Cu")
 		(at 170.75 19.83 180)
-		(descr "USB Type C, right-angle, SMT, https://datasheet.lcsc.com/szlcsc/1811141824_XKB-Enterprise-U262-161N-4BVC11_C319148.pdf")
+		(descr "USB Type C, right-angle, SMT, https://datasheet.lcsc.com/lcsc/2204071530_G-Switch-GT-USB-7010ASV_C2988369.pdf")
 		(tags "USB C Type-C Receptacle SMD")
 		(property "Reference" "J1"
-			(at 0 -5.715 180)
+			(at 0 -5.5 180)
 			(layer "F.SilkS")
 			(effects
@@
 		)
 		(property "Value" "USB_C_Receptacle_USB2.0_16P"
-			(at 0 4.935 180)
+			(at 0 5 180)
 			(layer "F.Fab")
 			(effects
@@
 		)
 		(fp_line
-			(start 5.32 -4.75)
+			(start 5.32 -4.85)
 			(end 5.32 4.18)
 			(stroke
@@
 		(fp_line
 			(start -5.32 4.18)
-			(end -5.32 -4.75)
+			(end -5.32 -4.85)
 			(stroke
 				(width 0.05)
@@
 		)
 		(fp_line
-			(start -5.32 -4.75)
-			(end 5.32 -4.75)
+			(start -5.32 -4.85)
+			(end 5.32 -4.85)
 			(stroke
 				(width 0.05)
@@
 		)
 		(pad "A1" smd rect
-			(at -3.35 -3.67 180)
-			(size 0.3 1.15)
+			(at -3.2 -3.725 180)
+			(size 0.6 1.24)
 			(layers "F.Cu" "F.Mask" "F.Paste")
 			(net 2 "GND")
@@
 		)
 		(pad "A4" smd rect
-			(at -2.55 -3.67 180)
-			(size 0.3 1.15)
+			(at -2.4 -3.725 180)
+			(size 0.6 1.24)
 			(layers "F.Cu" "F.Mask" "F.Paste")
 			(net 38 "+5V")
@@
 		)
 		(pad "A5" smd rect
-			(at -1.25 -3.67 180)
-			(size 0.3 1.15)
+			(at -1.25 -3.725 180)
+			(size 0.3 1.24)
 			(layers "F.Cu" "F.Mask" "F.Paste")
 			(net 39 "Net-(J1-CC1)")
@@
 		)
 		(pad "A6" smd rect
-			(at -0.25 -3.67 180)
-			(size 0.3 1.15)
+			(at -0.25 -3.725 180)
+			(size 0.3 1.24)
 			(layers "F.Cu" "F.Mask" "F.Paste")
 			(net 3 "D+")
@@
 		)
 		(pad "A7" smd rect
-			(at 0.25 -3.67 180)
-			(size 0.3 1.15)
+			(at 0.25 -3.725 180)
+			(size 0.3 1.24)
 			(layers "F.Cu" "F.Mask" "F.Paste")
 			(net 4 "D-")
@@
 		)
 		(pad "A8" smd rect
-			(at 1.25 -3.67 180)
-			(size 0.3 1.15)
+			(at 1.25 -3.725 180)
+			(size 0.3 1.24)
 			(layers "F.Cu" "F.Mask" "F.Paste")
 			(net 35 "unconnected-(J1-SBU1-PadA8)")
@@
 		)
 		(pad "A9" smd rect
-			(at 2.55 -3.67 180)
-			(size 0.3 1.15)
+			(at 2.4 -3.725 180)
+			(size 0.6 1.24)
 			(layers "F.Cu" "F.Mask" "F.Paste")
 			(net 38 "+5V")
@@
 		)
 		(pad "A12" smd rect
-			(at 3.35 -3.67 180)
-			(size 0.3 1.15)
+			(at 3.2 -3.725 180)
+			(size 0.6 1.24)
 			(layers "F.Cu" "F.Mask" "F.Paste")
 			(net 2 "GND")
@@
 		)
 		(pad "B1" smd rect
-			(at 3.05 -3.67 180)
-			(size 0.3 1.15)
+			(at 3.2 -3.725 180)
+			(size 0.6 1.24)
 			(layers "F.Cu" "F.Mask" "F.Paste")
 			(net 2 "GND")
@@
 		)
 		(pad "B4" smd rect
-			(at 2.25 -3.67 180)
-			(size 0.3 1.15)
+			(at 2.4 -3.725 180)
+			(size 0.6 1.24)
 			(layers "F.Cu" "F.Mask" "F.Paste")
 			(net 38 "+5V")
@@
 		)
 		(pad "B5" smd rect
-			(at 1.75 -3.67 180)
-			(size 0.3 1.15)
+			(at 1.75 -3.725 180)
+			(size 0.3 1.24)
 			(layers "F.Cu" "F.Mask" "F.Paste")
 			(net 37 "/CC2")
@@
 		)
 		(pad "B6" smd rect
-			(at 0.75 -3.67 180)
-			(size 0.3 1.15)
+			(at 0.75 -3.725 180)
+			(size 0.3 1.24)
 			(layers "F.Cu" "F.Mask" "F.Paste")
 			(net 3 "D+")
@@
 		)
 		(pad "B7" smd rect
-			(at -0.75 -3.67 180)
-			(size 0.3 1.15)
+			(at -0.75 -3.725 180)
+			(size 0.3 1.24)
 			(layers "F.Cu" "F.Mask" "F.Paste")
 			(net 4 "D-")
@@
 		)
 		(pad "B8" smd rect
-			(at -1.75 -3.67 180)
-			(size 0.3 1.15)
+			(at -1.75 -3.725 180)
+			(size 0.3 1.24)
 			(layers "F.Cu" "F.Mask" "F.Paste")
 			(net 36 "unconnected-(J1-SBU2-PadB8)")
@@
 		)
 		(pad "B9" smd rect
-			(at -2.25 -3.67 180)
-			(size 0.3 1.15)
+			(at -2.4 -3.725 180)
+			(size 0.6 1.24)
 			(layers "F.Cu" "F.Mask" "F.Paste")
 			(net 38 "+5V")
@@
 		)
 		(pad "B12" smd rect
-			(at -3.05 -3.67 180)
-			(size 0.3 1.15)
+			(at -3.2 -3.725 180)
+			(size 0.6 1.24)
 			(layers "F.Cu" "F.Mask" "F.Paste")
 			(net 2 "GND")
@@
 		)
 		(pad "S1" thru_hole oval
-			(at -4.32 -3.105 180)
+			(at -4.32 -3.125 180)
 			(size 1 2.1)
 			(drill oval 0.6 1.7)
@@
 		(pad "S1" thru_hole oval
 			(at -4.32 1.075 180)
-			(size 1 1.6)
-			(drill oval 0.6 1.2)
+			(size 1 1.8)
+			(drill oval 0.6 1.4)
 			(property pad_prop_heatsink)
 			(layers "*.Cu" "*.Mask")
@@
 		)
 		(pad "S1" thru_hole oval
-			(at 4.32 -3.105 180)
+			(at 4.32 -3.125 180)
 			(size 1 2.1)
 			(drill oval 0.6 1.7)
@@
 		(pad "S1" thru_hole oval
 			(at 4.32 1.075 180)
-			(size 1 1.6)
-			(drill oval 0.6 1.2)
+			(size 1 1.8)
+			(drill oval 0.6 1.4)
 			(property pad_prop_heatsink)
 			(layers "*.Cu" "*.Mask")
@@
 		)
 		(embedded_fonts no)
-		(model "${KICAD9_3DMODEL_DIR}/Connector_USB.3dshapes/USB_C_Receptacle_XKB_U262-16XN-4BVC11.step"
+		(model "${KICAD9_3DMODEL_DIR}/Connector_USB.3dshapes/USB_C_Receptacle_G-Switch_GT-USB-7010ASV.step"
 			(offset
 				(xyz 0 0 0)
@@
 			)
 		)
-		(property "Value" "R5.1kΩ"
+		(property "Value" "R5.1k"
 			(at 0 -1.43 90)
 			(layer "B.Fab")
@@
 			)
 		)
-		(property "Value" "100kΩ"
+		(property "Value" "100k"
 			(at 0 -1.43 0)
 			(layer "B.Fab")
@@
 			)
 		)
-		(property "Value" "100kΩ"
+		(property "Value" "100k"
 			(at 0 -1.43 0)
 			(layer "B.Fab")
@@
 		)
 	)
-	(footprint "Capacitor_SMD:C_0805_2012Metric_Pad1.18x1.45mm_HandSolder"
+	(footprint "Capacitor_SMD:C_0603_1608Metric_Pad1.08x0.95mm_HandSolder"
 		(layer "B.Cu")
 		(at 136.8 19.9 180)
-		(descr "Capacitor SMD 0805 (2012 Metric), square (rectangular) end terminal, IPC-7351 nominal with elongated pad for handsoldering. (Body size source: IPC-SM-782 page 76, https://www.pcb-3d.com/wordpress/wp-content/uploads/ipc-sm-782a_amendment_1_and_2.pdf, https://docs.google.com/spreadsheets/d/1BsfQQcO9C6DZCsRaXUlFlo91Tg2WpOkGARC1WS5S8t0/edit?usp=sharing), generated with kicad-footprint-generator")
+		(descr "Capacitor SMD 0603 (1608 Metric), square (rectangular) end terminal, IPC-7351 nominal with elongated pad for handsoldering. (Body size source: IPC-SM-782 page 76, https://www.pcb-3d.com/wordpress/wp-content/uploads/ipc-sm-782a_amendment_1_and_2.pdf), generated with kicad-footprint-generator")
 		(tags "capacitor handsolder")
 		(property "Reference" "C5"
-			(at 0 1.68 0)
+			(at 0 1.43 0)
 			(layer "B.SilkS")
 			(effects
@@
 		)
 		(property "Value" "0.1uF"
-			(at 0 -1.68 0)
+			(at 0 -1.43 0)
 			(layer "B.Fab")
 			(effects
@@
 		(attr smd)
 		(fp_line
-			(start -0.261252 0.735)
-			(end 0.261252 0.735)
+			(start -0.146267 0.51)
+			(end 0.146267 0.51)
 			(stroke
 				(width 0.12)
@@
 		)
 		(fp_line
-			(start -0.261252 -0.735)
-			(end 0.261252 -0.735)
+			(start -0.146267 -0.51)
+			(end 0.146267 -0.51)
 			(stroke
 				(width 0.12)
@@
 		)
 		(fp_line
-			(start 1.88 0.98)
-			(end 1.88 -0.98)
+			(start 1.65 0.73)
+			(end 1.65 -0.73)
 			(stroke
 				(width 0.05)
@@
 		)
 		(fp_line
-			(start 1.88 -0.98)
-			(end -1.88 -0.98)
+			(start 1.65 -0.73)
+			(end -1.65 -0.73)
 			(stroke
 				(width 0.05)
@@
 		)
 		(fp_line
-			(start -1.88 0.98)
-			(end 1.88 0.98)
+			(start -1.65 0.73)
+			(end 1.65 0.73)
 			(stroke
 				(width 0.05)
@@
 		)
 		(fp_line
-			(start -1.88 -0.98)
-			(end -1.88 0.98)
+			(start -1.65 -0.73)
+			(end -1.65 0.73)
 			(stroke
 				(width 0.05)
@@
 		)
 		(fp_line
-			(start 1 0.625)
-			(end 1 -0.625)
+			(start 0.8 0.4)
+			(end 0.8 -0.4)
 			(stroke
 				(width 0.1)
@@
 		)
 		(fp_line
-			(start 1 -0.625)
-			(end -1 -0.625)
+			(start 0.8 -0.4)
+			(end -0.8 -0.4)
 			(stroke
 				(width 0.1)
@@
 		)
 		(fp_line
-			(start -1 0.625)
-			(end 1 0.625)
+			(start -0.8 0.4)
+			(end 0.8 0.4)
 			(stroke
 				(width 0.1)
@@
 		)
 		(fp_line
-			(start -1 -0.625)
-			(end -1 0.625)
+			(start -0.8 -0.4)
+			(end -0.8 0.4)
 			(stroke
 				(width 0.1)
@@
 			(effects
 				(font
-					(size 0.5 0.5)
-					(thickness 0.08)
+					(size 0.4 0.4)
+					(thickness 0.06)
 				)
 				(justify mirror)
@@
 		)
 		(pad "1" smd roundrect
-			(at -1.0375 0 180)
-			(size 1.175 1.45)
+			(at -0.8625 0 180)
+			(size 1.075 0.95)
 			(layers "B.Cu" "B.Mask" "B.Paste")
-			(roundrect_rratio 0.212766)
+			(roundrect_rratio 0.25)
 			(net 2 "GND")
 			(pintype "passive")
 		)
 		(pad "2" smd roundrect
-			(at 1.0375 0 180)
-			(size 1.175 1.45)
+			(at 0.8625 0 180)
+			(size 1.075 0.95)
 			(layers "B.Cu" "B.Mask" "B.Paste")
-			(roundrect_rratio 0.212766)
+			(roundrect_rratio 0.25)
 			(net 46 "Net-(U3-VAUX)")
 			(pintype "passive")
 		)
 		(embedded_fonts no)
-		(model "${KICAD9_3DMODEL_DIR}/Capacitor_SMD.3dshapes/C_0805_2012Metric.step"
+		(model "${KICAD9_3DMODEL_DIR}/Capacitor_SMD.3dshapes/C_0603_1608Metric.step"
 			(offset
 				(xyz 0 0 0)
@@
 			)
 		)
-		(property "Value" "15kΩ"
+		(property "Value" "15k"
 			(at 0 -1.43 90)
 			(layer "B.Fab")
@@
 			)
 		)
-		(property "Value" "120Ω"
+		(property "Value" "120"
 			(at 0 -1.43 0)
 			(layer "B.Fab")
@@
 			)
 		)
-		(property "Value" "10kΩ"
+		(property "Value" "10k"
 			(at 0 -1.43 90)
 			(layer "B.Fab")
@@
 			)
 		)
-		(property "Value" "R5.1kΩ"
+		(property "Value" "R5.1k"
 			(at 0 -1.43 90)
 			(layer "B.Fab")
@@
 			)
 		)
+	)
+	(zone
+		(net 0)
+		(net_name "")
+		(layers "F.Cu" "B.Cu")
+		(hatch edge 0.5)
+		(connect_pads
+			(clearance 0)
+		)
+		(min_thickness 0.25)
+		(filled_areas_thickness no)
+		(keepout
+			(tracks not_allowed)
+			(vias not_allowed)
+			(pads not_allowed)
+			(copperpour not_allowed)
+			(footprints allowed)
+		)
+		(placement
+			(enabled no)
+			(sheetname "/")
+		)
+		(fill
+			(thermal_gap 0.5)
+			(thermal_bridge_width 0.5)
+		)
+		(polygon
+			(pts
+				(xy 150.634 19.443) (xy 165.7216 19.443) (xy 165.7216 25.285) (xy 150.634 25.285)
+			)
+		)

Commit message: Refactor code structure for improved readability and maintainability
Routing:
- net +5V_Boost: track 24.8 -> 23.5 mm
Changed lines of the file:
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@@
 	(segment
 		(start 141.5 20.5)
-		(end 145.9 20.5)
+		(end 144.3625 20.5)
 		(width 0.2)
 		(layer "B.Cu")
@@
 	)
 	(segment
-		(start 145.95 20.55)
-		(end 154 28.6)
+		(start 152.4625 28.6)
+		(end 145.5 21.6375)
 		(width 0.2)
 		(layer "B.Cu")
@@
 	)
 	(segment
-		(start 145.5 21)
+		(start 144.3625 20.5)
 		(end 145.5 21.6375)
-		(width 0.2)
-		(layer "B.Cu")
-		(net 8)
-	)
-	(segment
-		(start 145.9 20.5)
-		(end 145.95 20.55)
 		(width 0.2)
 		(layer "B.Cu")
@@
 	)
 	(segment
-		(start 145.95 20.55)
-		(end 145.5 21)
+		(start 134.85 22.05)
+		(end 135.4 21.5)
 		(width 0.2)
 		(layer "B.Cu")
@@
 	)
 	(segment
-		(start 134.85 22.05)
-		(end 135.4 21.5)
+		(start 154 28.6)
+		(end 152.4625 28.6)
 		(width 0.2)
 		(layer "B.Cu")

Commit message: firmware
Connections:
- C3 pad 1: VBAT -> 3.3V
- L1 pad 1: VBAT -> 3.3V
- U3 pad 5: VBAT -> 3.3V
- U3 pad 7: VBAT -> 3.3V
- U3 pad 8: VBAT -> 3.3V
Routing:
- net VBAT: track 103.6 -> 58.3 mm, vias 5 -> 1
- net 3.3V: track 32.0 -> 60.7 mm, vias 0 -> 2
- net +5V: track 45.9 -> 45.2 mm
